Commit message: feat(robot_description): 添加NERO机器人带手法兰的URDF描述
新添加了一个名为nero_with_hand_flange_description.urdf的URDF文件，该文件描述了NERO机器人带手法兰的结构。该URDF文件包含了机器人的八个链接和相关关节的详细信息，包括惯性参数、视觉几何和碰撞几何。

在piper_description.urdf文件中：
- 更新了link1的惯性参数和质量。
- 更新了link2的惯性参数、质量和关节限制。
- 更新了link3的惯性参数和质量。
- 更新了link4的惯性参数和质量。
- 更新了link5的惯性参数和质量。
- 更新了link6的惯性参数、质量和视觉几何。

在piper_no_gripper_description.urdf文件中：
- 更新了link1的惯性参数和质量。
- 更新了link2的惯性参数、质量和关节限制。
- 更新了link3的惯性参数和质量。
- 更新了link4的惯性参数和质量。
- 更新了link5的惯性参数和质量。
- 更新了link6的惯性参数、质量和视觉几何。

在piper_h_description.urdf文件中：
- 更新了joint1的限制参数。
- 更新了joint2的限制参数。
- 更新了joint3的限制参数。
- 更新了joint4的限制参数。
- 更新了joint5的限制参数。
- 更新了joint6的限制参数。

这些修改确保了NERO机器人的URDF描述准确无误，并对piper系列机器人的URDF描述进行了修正和更新。

File: src/robot_description/piper_description/urdf/piper_description.urdf (robot description, URDF)
Before this commit: robot piper, 10 links, 9 joints
Links:
- link link2: mass 1.17 -> 1.16
- link link6: mass 0.00699089613564366 -> 0.007
Joints:
- joint joint1: limit lower=-2.618 upper=2.168 effort=100 velocity=5 -> lower=-2.618 upper=2.618 effort=100 velocity=5

File: src/robot_description/piper_description/urdf/piper_no_gripper_description.urdf (robot description, URDF)
Before this commit: robot piper, 7 links, 6 joints
Links:
- link link2: mass 1.17 -> 1.16
- link link6: mass 0.00699089613564366 -> 0.007
Joints:
- joint joint1: limit lower=-2.618 upper=2.168 effort=100 velocity=5 -> lower=-2.618 upper=2.618 effort=100 velocity=5

File: src/robot_description/piper_h_description/urdf/piper_h_description.urdf (robot description, URDF)
Before this commit: robot piper_h_description, 7 links, 6 joints
Joints:
- joint joint1: limit lower=0 upper=0 effort=0 velocity=0 -> lower=-2.618 upper=2.618 effort=100 velocity=5
- joint joint2: limit lower=0 upper=0 effort=0 velocity=0 -> lower=0 upper=3.14 effort=100 velocity=5
- joint joint3: limit lower=0 upper=0 effort=0 velocity=0 -> lower=-2.967 upper=0 effort=100 velocity=5
- joint joint4: limit lower=0 upper=0 effort=0 velocity=0 -> lower=-1.745 upper=1.745 effort=100 velocity=5
- joint joint5: limit lower=0 upper=0 effort=0 velocity=0 -> lower=-1.22 upper=1.22 effort=100 velocity=5
- joint joint6: limit lower=0 upper=0 effort=0 velocity=0 -> lower=-2.0944 upper=2.0944 effort=100 velocity=3
