Commit message: fix(robot_description): 修正关节轴方向错误
关节 `link4` 到 `link5` 的轴方向从 `0 0 -1` 更改为 `0 0 1`，以确保关节运动方向正确。此修改涉及多个 URDF 文件中的相同部分，具体如下：

- 在 `piper_h_description.urdf` 中，`<joint name="joint4_5">` 的 `<axis>` 标签从 `xyz="0 0 -1"` 更改为 `xyz="0 0 1"`。
- 在 `piper_h_description_d435.urdf` 中，`<joint name="joint4_5">` 的 `<axis>` 标签从 `xyz="0 0 -1"` 更改为 `xyz="0 0 1"`。
- 在 `piper_h_description_d435_dark.urdf` 中，`<joint name="joint4_5">` 的 `<axis>` 标签从 `xyz="0 0 -1"` 更改为 `xyz="0 0 1"`。
- 在 `piper_h_description_dark.urdf` 中，`<joint name="joint4_5">` 的 `<axis>` 标签从 `xyz="0 0 -1"` 更改为 `xyz="0 0 1"`。

这些更改确保了关节在模拟和实际操作中的运动方向一致。

File: src/robot_description/piper_h_description/urdf/piper_h_description.urdf (robot description, URDF)
Before this commit: robot piper_h_description, 7 links, 6 joints
Joints:
- joint joint5: axis 0 0 -1 -> 0 0 1

File: src/robot_description/piper_h_description/urdf/piper_h_description_d435.urdf (robot description, URDF)
Before this commit: robot piper_l_camera, 13 links, 12 joints
Joints:
- joint joint5: axis 0 0 -1 -> 0 0 1

File: src/robot_description/piper_h_description/urdf/piper_h_description_d435_dark.urdf (robot description, URDF)
Before this commit: robot piper_l_camera, 13 links, 12 joints
Joints:
- joint joint5: axis 0 0 -1 -> 0 0 1

File: src/robot_description/piper_h_description/urdf/piper_h_description_dark.urdf (robot description, URDF)
Before this commit: robot piper_h_description, 7 links, 6 joints
Joints:
- joint joint5: axis 0 0 -1 -> 0 0 1
